File: hardware/encoder_no_switch.kicad_sch (KiCad schematic)
At the start: 7 parts

Commit message: harware v1 done
Parts:
- gave numbers to parts that had none: 7
Changed lines of the file:
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@@
   (symbol (lib_id "Device:C") (at 151.13 102.87 0)
     (in_bom yes) (on_board yes)
-    (property "Reference" "C?" (id 0) (at 154.051 101.7016 0)
+    (property "Reference" "C2" (id 0) (at 154.051 101.7016 0)
       (effects (font (size 1.27 1.27)) (justify left))
     )
@@
   (symbol (lib_id "Device:R") (at 120.65 101.6 0)
     (in_bom yes) (on_board yes)
-    (property "Reference" "R?" (id 0) (at 122.428 100.4316 0)
+    (property "Reference" "R2" (id 0) (at 122.428 100.4316 0)
       (effects (font (size 1.27 1.27)) (justify left))
     )
@@
   (symbol (lib_id "power:GND") (at 151.13 114.3 0)
     (in_bom yes) (on_board yes)
-    (property "Reference" "#PWR?" (id 0) (at 151.13 120.65 0)
+    (property "Reference" "#PWR0110" (id 0) (at 151.13 120.65 0)
       (effects (font (size 1.27 1.27)) hide)
     )
@@
   (symbol (lib_id "Device:R") (at 116.84 95.25 270)
     (in_bom yes) (on_board yes)
-    (property "Reference" "R?" (id 0) (at 116.84 89.9922 90))
+    (property "Reference" "R1" (id 0) (at 116.84 89.9922 90))
     (property "Value" "10k" (id 1) (at 116.84 92.3036 90))
     (property "Footprint" "Resistor_SMD:R_0603_1608Metric" (id 2) (at 116.84 93.472 90)
@@
   (symbol (lib_id "Device:Rotary_Encoder") (at 130.81 81.28 90)
     (in_bom yes) (on_board yes)
-    (property "Reference" "SW?" (id 0) (at 131.0894 75.438 90)
+    (property "Reference" "SW1" (id 0) (at 131.0894 75.438 90)
       (effects (font (size 1.27 1.27)) (justify right))
     )
@@
   (symbol (lib_id "Device:C") (at 111.76 105.41 0)
     (in_bom yes) (on_board yes)
-    (property "Reference" "C?" (id 0) (at 114.681 104.2416 0)
+    (property "Reference" "C1" (id 0) (at 114.681 104.2416 0)
       (effects (font (size 1.27 1.27)) (justify left))
     )
@@
   (symbol (lib_id "power:GND") (at 111.76 114.3 0)
     (in_bom yes) (on_board yes)
-    (property "Reference" "#PWR?" (id 0) (at 111.76 120.65 0)
+    (property "Reference" "#PWR0111" (id 0) (at 111.76 120.65 0)
       (effects (font (size 1.27 1.27)) hide)
     )
@@
   (symbol (lib_id "Device:R") (at 140.97 101.6 0)
     (in_bom yes) (on_board yes)
-    (property "Reference" "R?" (id 0) (at 142.748 100.4316 0)
+    (property "Reference" "R3" (id 0) (at 142.748 100.4316 0)
       (effects (font (size 1.27 1.27)) (justify left))
     )
@@
   (symbol (lib_id "power:+3.3V") (at 130.81 107.95 180)
     (in_bom yes) (on_board yes)
-    (property "Reference" "#PWR?" (id 0) (at 130.81 104.14 0)
+    (property "Reference" "#PWR0112" (id 0) (at 130.81 104.14 0)
       (effects (font (size 1.27 1.27)) hide)
     )
@@
   (symbol (lib_id "power:GND") (at 130.81 99.06 0)
     (in_bom yes) (on_board yes)
-    (property "Reference" "#PWR?" (id 0) (at 130.81 105.41 0)
+    (property "Reference" "#PWR0113" (id 0) (at 130.81 105.41 0)
       (effects (font (size 1.27 1.27)) hide)
     )
@@
   (symbol (lib_id "Device:R") (at 146.05 93.98 270)
     (in_bom yes) (on_board yes)
-    (property "Reference" "R?" (id 0) (at 146.05 88.7222 90))
+    (property "Reference" "R4" (id 0) (at 146.05 88.7222 90))
     (property "Value" "10k" (id 1) (at 146.05 91.0336 90))
     (property "Footprint" "Resistor_SMD:R_0603_1608Metric" (id 2) (at 146.05 92.202 90)

Commit message: up
Parts:
- renumbered C1 to C5, C2 to C6, R2 to R10, R3 to R11, R4 to R12, R1 to R9, SW1 to SW3
Changed lines of the file:
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@@
   (symbol (lib_id "Device:C") (at 151.13 102.87 0)
     (in_bom yes) (on_board yes)
-    (property "Reference" "C2" (id 0) (at 154.051 101.7016 0)
+    (property "Reference" "C6" (id 0) (at 154.051 101.7016 0)
       (effects (font (size 1.27 1.27)) (justify left))
     )
@@
   (symbol (lib_id "Device:R") (at 120.65 101.6 0)
     (in_bom yes) (on_board yes)
-    (property "Reference" "R2" (id 0) (at 122.428 100.4316 0)
+    (property "Reference" "R10" (id 0) (at 122.428 100.4316 0)
       (effects (font (size 1.27 1.27)) (justify left))
     )
@@
   (symbol (lib_id "power:GND") (at 151.13 114.3 0)
     (in_bom yes) (on_board yes)
-    (property "Reference" "#PWR0110" (id 0) (at 151.13 120.65 0)
+    (property "Reference" "#PWR0118" (id 0) (at 151.13 120.65 0)
       (effects (font (size 1.27 1.27)) hide)
     )
@@
   (symbol (lib_id "Device:R") (at 116.84 95.25 270)
     (in_bom yes) (on_board yes)
-    (property "Reference" "R1" (id 0) (at 116.84 89.9922 90))
+    (property "Reference" "R9" (id 0) (at 116.84 89.9922 90))
     (property "Value" "10k" (id 1) (at 116.84 92.3036 90))
     (property "Footprint" "Resistor_SMD:R_0603_1608Metric" (id 2) (at 116.84 93.472 90)
@@
   (symbol (lib_id "Device:Rotary_Encoder") (at 130.81 81.28 90)
     (in_bom yes) (on_board yes)
-    (property "Reference" "SW1" (id 0) (at 131.0894 75.438 90)
+    (property "Reference" "SW3" (id 0) (at 131.0894 75.438 90)
       (effects (font (size 1.27 1.27)) (justify right))
     )
@@
   (symbol (lib_id "Device:C") (at 111.76 105.41 0)
     (in_bom yes) (on_board yes)
-    (property "Reference" "C1" (id 0) (at 114.681 104.2416 0)
+    (property "Reference" "C5" (id 0) (at 114.681 104.2416 0)
       (effects (font (size 1.27 1.27)) (justify left))
     )
@@
   (symbol (lib_id "power:GND") (at 111.76 114.3 0)
     (in_bom yes) (on_board yes)
-    (property "Reference" "#PWR0111" (id 0) (at 111.76 120.65 0)
+    (property "Reference" "#PWR0119" (id 0) (at 111.76 120.65 0)
       (effects (font (size 1.27 1.27)) hide)
     )
@@
   (symbol (lib_id "Device:R") (at 140.97 101.6 0)
     (in_bom yes) (on_board yes)
-    (property "Reference" "R3" (id 0) (at 142.748 100.4316 0)
+    (property "Reference" "R11" (id 0) (at 142.748 100.4316 0)
       (effects (font (size 1.27 1.27)) (justify left))
     )
@@
   (symbol (lib_id "power:+3.3V") (at 130.81 107.95 180)
     (in_bom yes) (on_board yes)
-    (property "Reference" "#PWR0112" (id 0) (at 130.81 104.14 0)
+    (property "Reference" "#PWR0120" (id 0) (at 130.81 104.14 0)
       (effects (font (size 1.27 1.27)) hide)
     )
@@
   (symbol (lib_id "power:GND") (at 130.81 99.06 0)
     (in_bom yes) (on_board yes)
-    (property "Reference" "#PWR0113" (id 0) (at 130.81 105.41 0)
+    (property "Reference" "#PWR0121" (id 0) (at 130.81 105.41 0)
       (effects (font (size 1.27 1.27)) hide)
     )
@@
   (symbol (lib_id "Device:R") (at 146.05 93.98 270)
     (in_bom yes) (on_board yes)
-    (property "Reference" "R4" (id 0) (at 146.05 88.7222 90))
+    (property "Reference" "R12" (id 0) (at 146.05 88.7222 90))
     (property "Value" "10k" (id 1) (at 146.05 91.0336 90))
     (property "Footprint" "Resistor_SMD:R_0603_1608Metric" (id 2) (at 146.05 92.202 90)
